File: nRF_touch.brd (EAGLE design)
At the start: 46.5 x 82.2 mm, 87 parts, among them IC1 MCP73831/OT, Q1 BSS138BKW, T1 BSS84, T2 BC847, T3 BC847, T4 BC847, U1 ADP160, U2 AT42QT1040, Y1 32.768kHz, Y2 32MHz-3.2X2.5

Commit message: Routing complete
Parts:
- moved R5 0.51 mm to (9.29, 46.8)
- moved L1 0.13 mm to (24.4, 76.5)
Routing:
- net GND: track 74.7 -> 42.5 mm, vias 10 -> 6
- net VCC: track 74.4 -> 50.8 mm, vias 12 -> 10
- net AT42_COUT: track 91.3 -> 109.2 mm, vias 6 -> 3
- net SPIM_DIN: track 40.8 -> 43.6 mm, vias 1 -> 2
- net EXTMODE: track 1.86 -> 4.41 mm
- net NEO_PIN: track 36.1 -> 33.8 mm
- net AT42_GOUT: track 29.5 -> 28.4 mm

Commit message: Added resistors Routing optimized
Parts:
- added R20: 47k, SparkFun-Resistors:0603
- added R21: 100k, SparkFun-Resistors:0603
- added R22, R23: 10k, SparkFun-Resistors:0603
- added RX: TESTPOINT_22, test_points:TESTPOINT_22
- moved C21 5.93 mm to (26.2, 49.8), turned to 180 degrees
- moved R3 5.53 mm to (31.8, 13.3), turned to 180 degrees
- moved C20 4.85 mm to (26.2, 47.4), turned to 180 degrees
- moved Y1 1.85 mm to (29.0, 48.5), turned to 270 degrees
- moved SWDCLK 1.09 mm to (35.9, 30.9)
- moved T3 1.02 mm to (34.2, 15.4)
- moved R5 0.92 mm to (10.2, 47.0)
- moved SWDIO 0.64 mm to (34.7, 33.0)
- moved C8 0.51 mm to (3.17, 68.8)
- moved R1 0.46 mm to (15.4, 65.0), turned to 270 degrees
- moved C5 0.40 mm to (21.7, 68.1)
- moved C3 0.38 mm to (21.7, 65.3)
Connections:
- removed net N$10: R3.2, U$1.P$2, U$7.P$2
- removed net N$31: U$6.8
- new net N$23: R3.2, T3.3
- new net PIN_BCK: R21.1, U$6.10
- new net RX: RX.P$1, U$6.15
- net CHRG_END: now also U$6.8; no longer U$6.43
- net GND: now also R20.2
- net LED_BCK: now also R21.2; no longer U$6.10
- net N$13: now also R3.1; no longer T3.3
- net SCL: now also R23.2
- net SDA: now also R22.2
- net SW_POWER: now also R20.1
- net VCC: now also R22.1, R23.1, U$1.P$2, U$7.P$2; no longer R3.1
Routing:
- net GND: track 42.5 -> 100.3 mm, vias 6 -> 16
- net N$10: track 29.9 -> 0.00 mm, vias 2 -> 0
- net PIN_BCK: track 0.00 -> 9.65 mm
- net LED_BCK: track 71.0 -> 62.2 mm
- net VCC: track 50.8 -> 58.5 mm, vias 10 -> 11
- net SW_POWER: track 22.9 -> 29.9 mm, vias 2 -> 3
- net N$13: track 27.8 -> 24.6 mm, vias 2 -> 3
- net RX: track 0.00 -> 2.75 mm
- net N$25: track 8.86 -> 11.6 mm
- net N$23: track 0.00 -> 2.46 mm
- net SCL: track 83.1 -> 85.3 mm
- net SDA: track 74.7 -> 76.8 mm
- net N$16: track 7.02 -> 4.92 mm
- net AT42_COUT: track 109.2 -> 107.5 mm
- net CPAD: track 11.8 -> 13.3 mm
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- added copper zone on layer 16, net N$26
Other:
- outline, holes or cut-outs redrawn

Commit message: Errors corrected #1
Parts:
- removed U3: (no value), adafruit:FGPMMOPA6H
- moved R5 2.41 mm to (12.6, 47.0)
- moved R6 2.41 mm to (15.5, 42.0)
- moved R7 2.41 mm to (14.6, 44.6)
- moved U$4 2.41 mm to (8.57, 42.2)
- moved C1 2.41 mm to (16.4, 44.6)
- moved C4 0.25 mm to (20.4, 17.0)
Routing:
- net SPIM_SCK: track 44.4 -> 45.7 mm
- net GND: track 100.3 -> 100.9 mm
Other:
- board size 46.5 x 82.2 mm -> 46.5 x 82.7 mm

Commit message: Smashing
Parts:
- moved C23 0.36 mm to (27.9, 28.4)
- moved C22 0.25 mm to (24.0, 31.9)
- moved R1 0.13 mm to (15.2, 65.0)

Commit message: Screen hole
Routing:
- net SPIM_DO: track 38.5 -> 35.9 mm
- net 5150_CS: track 49.4 -> 47.6 mm
- net VBAT: track 73.8 -> 72.1 mm
- net SHARP_CS: track 35.3 -> 33.9 mm
Other:
- outline, holes or cut-outs redrawn
Changed lines of the file:
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@@
 <wire x1="18.923" y1="74.0156" x2="18.415" y2="73.65" width="0" layer="20"/>
 <wire x1="18.415" y1="73.65" x2="-0.127" y2="73.65" width="0" layer="20"/>
-<wire x1="-0.127" y1="73.65" x2="-0.127" y2="0" width="0" layer="20"/>
+<wire x1="-0.127" y1="73.65" x2="0" y2="47.625" width="0" layer="20"/>
+<wire x1="0" y1="47.625" x2="1.778" y2="46.482" width="0" layer="20"/>
+<wire x1="1.778" y1="46.482" x2="1.778" y2="37.846" width="0" layer="20"/>
+<wire x1="1.778" y1="37.846" x2="0" y2="36.449" width="0" layer="20"/>
+<wire x1="0" y1="36.449" x2="-0.127" y2="0" width="0" layer="20"/>
 <rectangle x1="41.529" y1="18.669" x2="47.625" y2="46.101" layer="41"/>
 <rectangle x1="41.529" y1="18.669" x2="47.625" y2="46.101" layer="42"/>
@@
 <wire x1="26.67" y1="36.83" x2="29.997" y2="36.83" width="0.1778" layer="16"/>
 <wire x1="29.997" y1="36.83" x2="30" y2="36.827" width="0.1778" layer="16"/>
-<wire x1="11.692" y1="40.54" x2="3.964" y2="40.54" width="0.1778" layer="16"/>
-<wire x1="3.964" y1="40.54" x2="3.683" y2="40.259" width="0.1778" layer="16"/>
-<wire x1="3.683" y1="40.259" x2="3.683" y2="36.703" width="0.1778" layer="16"/>
-<wire x1="3.683" y1="36.703" x2="4.953" y2="35.433" width="0.1778" layer="16"/>
+<wire x1="11.692" y1="40.54" x2="6.504" y2="40.54" width="0.1778" layer="16"/>
+<wire x1="6.504" y1="40.54" x2="4.953" y2="38.989" width="0.1778" layer="16"/>
+<wire x1="4.953" y1="38.989" x2="4.953" y2="36.322" width="0.1778" layer="16"/>
+<wire x1="4.953" y1="36.322" x2="4.953" y2="35.433" width="0.1778" layer="16"/>
 <wire x1="4.953" y1="35.433" x2="4.953" y2="32.766" width="0.1778" layer="16"/>
 <wire x1="4.953" y1="32.766" x2="4.064" y2="31.877" width="0.1778" layer="16"/>
@@
 <wire x1="27.559" y1="37.592" x2="29.965" y2="37.592" width="0.1778" layer="16"/>
 <wire x1="29.965" y1="37.592" x2="30" y2="37.627" width="0.1778" layer="16"/>
-<wire x1="3.048" y1="33.909" x2="3.048" y2="40.64" width="0.1778" layer="16"/>
-<wire x1="3.048" y1="40.64" x2="3.429" y2="41.021" width="0.1778" layer="16"/>
-<wire x1="3.429" y1="41.021" x2="11.673" y2="41.021" width="0.1778" layer="16"/>
 <wire x1="11.673" y1="41.021" x2="11.692" y2="41.04" width="0.1778" layer="16"/>
-<wire x1="13.951" y1="41.04" x2="11.692" y2="41.04" width="0.1778" layer="16"/>
+<wire x1="11.77971875" y1="41.04" x2="13.951" y2="41.04" width="0.1778" layer="16"/>
+<wire x1="11.77971875" y1="41.04" x2="11.692" y2="41.04" width="0.1778" layer="16"/>
+<wire x1="3.048" y1="33.909" x2="3.048" y2="35.052" width="0.1778" layer="16"/>
+<wire x1="3.048" y1="35.052" x2="4.318" y2="36.322" width="0.1778" layer="16"/>
+<wire x1="4.318" y1="36.322" x2="4.318" y2="39.37" width="0.1778" layer="16"/>
+<wire x1="4.318" y1="39.37" x2="5.969" y2="41.021" width="0.1778" layer="16"/>
+<wire x1="5.969" y1="41.021" x2="11.76071875" y2="41.021" width="0.1778" layer="16"/>
+<wire x1="11.76071875" y1="41.021" x2="11.77971875" y2="41.04" width="0.1778" layer="16"/>
 </signal>
 <signal name="EXTCOMM">
@@
 <wire x1="22.987" y1="38.862" x2="17.653" y2="38.862" width="0.1778" layer="1"/>
 <wire x1="17.653" y1="38.862" x2="14.732" y2="41.783" width="0.1778" layer="1"/>
-<wire x1="14.732" y1="41.783" x2="2.794" y2="41.783" width="0.1778" layer="1"/>
-<wire x1="2.794" y1="41.783" x2="1.524" y2="43.053" width="0.1778" layer="1"/>
-<wire x1="1.524" y1="43.053" x2="1.524" y2="60.706" width="0.1778" layer="1"/>
-<wire x1="1.524" y1="60.706" x2="2.159" y2="61.341" width="0.1778" layer="1"/>
+<wire x1="14.732" y1="41.783" x2="5.08" y2="41.783" width="0.1778" layer="1"/>
+<wire x1="5.08" y1="41.783" x2="4.191" y2="42.672" width="0.1778" layer="1"/>
+<wire x1="4.191" y1="42.672" x2="4.191" y2="56.769" width="0.1778" layer="1"/>
+<wire x1="4.191" y1="56.769" x2="2.159" y2="58.801" width="0.1778" layer="1"/>
+<wire x1="2.159" y1="58.801" x2="2.159" y2="61.341" width="0.1778" layer="1"/>
 </signal>
 <signal name="VBAT" class="1">
@@
 <wire x1="8.509" y1="60.452" x2="8.509" y2="61.5591" width="0.254" layer="16"/>
 <wire x1="8.509" y1="61.5591" x2="9.464" y2="62.1331" width="0.254" layer="16"/>
-<wire x1="0.762" y1="54.102" x2="0.762" y2="53.721" width="0.1778" layer="16"/>
-<wire x1="0.762" y1="56.642" x2="0.762" y2="54.102" width="0.1778" layer="16"/>
-<wire x1="2.159" y1="58.039" x2="0.762" y2="56.642" width="0.1778" layer="16"/>
-<wire x1="3.175" y1="58.039" x2="2.159" y2="58.039" width="0.1778" layer="16"/>
 <wire x1="3.175" y1="58.42" x2="3.175" y2="58.039" width="0.1778" layer="16"/>
 <wire x1="3.175" y1="58.42" x2="3.175" y2="58.508" width="0.1778" layer="16"/>
-<wire x1="0.762" y1="53.086" x2="0.762" y2="53.721" width="0.1778" layer="16"/>
-<wire x1="0.762" y1="43.307" x2="0.762" y2="53.086" width="0.1778" layer="16"/>
-<wire x1="0.762" y1="43.18" x2="0.762" y2="43.307" width="0.1778" layer="16"/>
-<wire x1="2.667" y1="41.275" x2="0.762" y2="43.18" width="0.1778" layer="1"/>
-<wire x1="10.541" y1="41.275" x2="2.667" y2="41.275" width="0.1778" layer="1"/>
 <wire x1="13.97" y1="37.846" x2="10.541" y2="41.275" width="0.1778" layer="1"/>
 <wire x1="14.351" y1="37.846" x2="13.97" y2="37.846" width="0.1778" layer="16"/>
@@
 <wire x1="22.987" y1="25.273" x2="22.606" y2="25.273" width="0.1778" layer="16"/>
 <wire x1="24.13" y1="25.273" x2="24.169" y2="25.273" width="0.1778" layer="16"/>
-<via x="0.762" y="43.18" extent="1-16" drill="0.3556"/>
 <via x="13.97" y="37.846" extent="1-16" drill="0.3556"/>
 <via x="16.002" y="31.877" extent="1-16" drill="0.3556"/>
@@
 <via x="22.606" y="25.273" extent="1-16" drill="0.3556"/>
 <wire x1="22.606" y1="25.273" x2="22.987" y2="25.273" width="0.1778" layer="16"/>
+<wire x1="4.318" y1="41.275" x2="3.556" y2="42.037" width="0.1778" layer="1"/>
+<wire x1="3.556" y1="42.037" x2="3.556" y2="52.197" width="0.1778" layer="1"/>
+<wire x1="3.556" y1="52.197" x2="1.905" y2="53.848" width="0.1778" layer="1"/>
+<wire x1="1.905" y1="53.848" x2="1.905" y2="54.737" width="0.1778" layer="1"/>
+<via x="1.905" y="54.737" extent="1-16" drill="0.35"/>
+<wire x1="1.905" y1="54.737" x2="1.905" y2="57.912" width="0.1778" layer="16"/>
+<wire x1="2.413" y1="58.42" x2="3.175" y2="58.42" width="0.1778" layer="16"/>
+<wire x1="10.541" y1="41.275" x2="4.318" y2="41.275" width="0.1778" layer="1"/>
+<wire x1="1.905" y1="57.912" x2="2.413" y2="58.42" width="0.1778" layer="16"/>
 </signal>
 <signal name="SW_POWER">
@@
 <wire x1="36.056" y1="37.211" x2="36.04" y2="37.227" width="0.1524" layer="16"/>
 <wire x1="5.654" y1="49.954" x2="4.869" y2="49.954" width="0.1524" layer="16"/>
-<wire x1="4.869" y1="49.954" x2="2.159" y2="47.244" width="0.1524" layer="16"/>
-<wire x1="2.159" y1="47.244" x2="2.159" y2="37.084" width="0.1524" layer="16"/>
-<wire x1="2.159" y1="37.084" x2="1.143" y2="36.068" width="0.1524" layer="16"/>
-<wire x1="1.143" y1="36.068" x2="1.143" y2="16.764" width="0.1524" layer="16"/>
+<wire x1="4.869" y1="49.954" x2="3.175" y2="48.26" width="0.1524" layer="16"/>
+<wire x1="3.175" y1="48.26" x2="3.175" y2="37.338" width="0.1524" layer="16"/>
+<wire x1="3.175" y1="37.338" x2="1.143" y2="35.306" width="0.1524" layer="16"/>
+<wire x1="1.143" y1="35.306" x2="1.143" y2="16.764" width="0.1524" layer="16"/>
 <wire x1="1.143" y1="16.764" x2="1.905" y2="16.002" width="0.1524" layer="16"/>
 <wire x1="1.905" y1="16.002" x2="7.747" y2="16.002" width="0.1524" layer="16"/>
